File: Panel/Panel Clean.kicad_pcb (KiCad board)
At the start: 2 copper layers, 70.8 x 128.5 mm, 28 parts

Commit message: Clean front panel changes
Other:
- net class Default removed
- board text added: "."
- board text added: ".."
- board text added: "..."
- board text added: "ACC"
- board text added: "CHAOS"
- board text added: "CLOCK"
- board text added: "FILL"
- board text added: "OUTPUTS"
- board text added: "RESET"
- board text added: "SPEED"
- board text added: "TAP"
- board text added: "TRIG"
- board text added: "triggerspace"
- board text removed: "ACC 1"
- board text removed: "ACC 2"
- board text removed: "ACC 3"
- board text removed: "CH 1"
- board text removed: "CH 2"
- board text removed: "CH 3"
- board text removed: "Clock"
- board text removed: "Fill 1"
- board text removed: "Fill 2"
- board text removed: "Fill 3"
- board text removed: "NanoGris"
- board text removed: "R N D"
- board text removed: "Random"
- board text removed: "Reset"
- board text removed: "Speed"
- board text removed: "Tap"
