File: NanoGris.kicad_pcb (KiCad board)
At the start: 2 copper layers, 164.6 x 108 mm, 112 parts, among them J10 Conn_01x12, J11 Conn_01x12, J12 Conn_02x05_Odd_Even, J13 Conn_01x10, J14 Conn_01x10, J15 Conn_01x10, J16 Conn_01x03, J7 Conn_01x10, Q1 2N3904, Q2 2N3904, U1 MCP6002_1, U2 MCP6002_1, U3 MCP6002_1, U4 L7805, U5 LM4040LP-5, U6 74HC595, X1 CV_X, Y1 CV_Y

Commit message: Updated with MIDI-TRS ports, numerous tweaks.
Moved front panel into main PCB design, remove old panels and gerbers that will no longer fit this design.
Parts:
- removed J16: Conn_01x03, Connector_PinHeader_2.54mm:PinHeader_1x03_P2.54mm_Vertical
- added ?: , , F.Cu at (68.5, 134.0)
- added ?: , , F.Cu at (15.0, 134.2)
- added ?: , , F.Cu at (68.4, 11.9)
- added ?: , , F.Cu at (15.5, 11.8)
- added C17: 100nf, Capacitor_THT:C_Disc_D5.0mm_W2.5mm_P2.50mm, F.Cu at (250.4, 70.9)
- added D7: 1n4148, Diode_THT:D_DO-34_SOD68_P7.62mm_Horizontal, B.Cu at (238.1, 44.7)
- added H1: MountingHole, MountingHole:MountingHole_6mm, F.Cu at (34.9, 120.7)
- added H10: MountingHole, MountingHole:MountingHole_6mm, F.Cu at (34.9, 25.5)
- added H11: MountingHole, MountingHole:MountingHole_6mm, F.Cu at (51.9, 97.9)
- added H12: MountingHole, MountingHole:MountingHole_6mm, F.Cu at (34.9, 38.2)
- added H13: MountingHole, MountingHole:MountingHole_6mm, F.Cu at (34.9, 97.9)
- added H14: MountingHole, MountingHole:MountingHole_6mm, F.Cu at (17.9, 67.4)
- added H15: MountingHole, MountingHole:MountingHole_6mm, F.Cu at (17.9, 97.9)
- added H16: MountingHole, MountingHole:MountingHole_6mm, F.Cu at (67.9, 97.9)
- added H17: MountingHole, MountingHole:MountingHole_6mm, F.Cu at (35.0, 52.7)
- added H18: MountingHole, MountingHole:MountingHole_3mm, F.Cu at (34.8, 69.8)
- added H19: MountingHole, MountingHole:MountingHole_3mm, F.Cu at (67.8, 69.8)
- added H2: MountingHole, MountingHole:MountingHole_6mm, F.Cu at (34.9, 109.3)
- added H20: MountingHole, MountingHole:MountingHole_3mm, F.Cu at (51.5, 69.8)
- added H21: MountingHole, MountingHole:MountingHole_3mm, F.Cu at (52.3, 38.1)
- added H22: MountingHole, MountingHole:MountingHole_8.4mm_M8, F.Cu at (17.9, 25.5)
- added H23: MountingHole, MountingHole:MountingHole_8.4mm_M8, F.Cu at (34.9, 82.6)
- added H24: MountingHole, MountingHole:MountingHole_8.4mm_M8, F.Cu at (17.9, 82.6)
- added H25: MountingHole, MountingHole:MountingHole_8.4mm_M8, F.Cu at (17.9, 52.1)
- added H26: MountingHole, MountingHole:MountingHole_8.4mm_M8, F.Cu at (51.9, 82.6)
- added H27: MountingHole, MountingHole:MountingHole_8.4mm_M8, F.Cu at (67.9, 82.6)
- added H28: MountingHole, MountingHole:MountingHole_8.4mm_M8, F.Cu at (52.3, 25.5)
- added H3: MountingHole, MountingHole:MountingHole_6mm, F.Cu at (67.9, 109.3)
- added H4: MountingHole, MountingHole:MountingHole_6mm, F.Cu at (17.9, 109.3)
- added H5: MountingHole, MountingHole:MountingHole_6mm, F.Cu at (67.9, 52.8)
- added H5: MountingHole, MountingHole:MountingHole_6mm, F.Cu at (51.9, 109.3)
- added H5: MountingHole, MountingHole:MountingHole_6mm, F.Cu at (52.1, 52.7)
- added H6: MountingHole, MountingHole:MountingHole_6mm, F.Cu at (51.9, 120.7)
- added H7: MountingHole, MountingHole:MountingHole_6mm, F.Cu at (67.9, 120.7)
- added H8: MountingHole, MountingHole:MountingHole_6mm, F.Cu at (17.9, 120.7)
- added H9: MountingHole, MountingHole:MountingHole_6mm, F.Cu at (17.9, 40.7)
- added J1: Conn_01x2, Connector_PinSocket_2.54mm:PinSocket_1x02_P2.54mm_Vertical, B.Cu at (125.2, 39.4)
- added J2: Conn_01x2, Connector_PinSocket_2.54mm:PinSocket_1x02_P2.54mm_Vertical, B.Cu at (150.6, 39.4)
- added J3: Conn_01x2, Connector_PinHeader_2.54mm:PinHeader_1x02_P2.54mm_Vertical, B.Cu at (257.9, 26.6)
- added J4: Conn_01x2, Connector_PinSocket_2.54mm:PinSocket_1x02_P2.54mm_Vertical, B.Cu at (107.8, 26.7)
- added JP1: SolderJumper_2_Bridged, Jumper:SolderJumper-2_P1.3mm_Bridged_RoundedPad1.0x1.5mm, F.Cu at (130.4, 40.6)
- added JP2: SolderJumper_2_Bridged, Jumper:SolderJumper-2_P1.3mm_Bridged_RoundedPad1.0x1.5mm, F.Cu at (118.3, 28.1)
- added MIDI_IN1: MIDI_IN, Connector_Audio:Jack_3.5mm_QingPu_WQP-PJ398SM_Vertical_CircularHoles, F.Cu at (242.2, 59.1)
- added MIDI_OUT1: MIDI_OUT, Connector_Audio:Jack_3.5mm_QingPu_WQP-PJ398SM_Vertical_CircularHoles, F.Cu at (257.9, 59.2)
- added R46: 4.7k, Resistor_THT:R_Axial_DIN0204_L3.6mm_D1.6mm_P7.62mm_Horizontal, B.Cu at (250.9, 64.6)
- added R47: 220, Resistor_THT:R_Axial_DIN0204_L3.6mm_D1.6mm_P7.62mm_Horizontal, F.Cu at (154.5, 44.9)
- added R48: 220, Resistor_THT:R_Axial_DIN0204_L3.6mm_D1.6mm_P7.62mm_Horizontal, B.Cu at (235.7, 56.1)
- added R49: 220, Resistor_THT:R_Axial_DIN0204_L3.6mm_D1.6mm_P7.62mm_Horizontal, B.Cu at (257.8, 44.9)
- added R50: 220, Resistor_THT:R_Axial_DIN0204_L3.6mm_D1.6mm_P7.62mm_Horizontal, B.Cu at (251.5, 52.1)
- added U8: 6N138, Package_DIP:DIP-8_W7.62mm_Socket_LongPads, B.Cu at (253.4, 75.1)
- D5, D6: value 1n4148 -> 1N5817
- FID2: moved to B.Cu
- moved FID2 32.5 mm to (252.5, 30.7), turned to 180 degrees
- moved RESET2 14.7 mm to (221.7, 50.4)
- moved C12 11.3 mm to (163.0, 76.4), turned to 0 degrees
- moved D4 5.01 mm to (241.1, 38.1)
- moved R42 4.75 mm to (157.2, 44.8)
- moved C11 3.99 mm to (154.2, 80.4), turned to -90 degrees
- moved U4 3.53 mm to (165.7, 80.5), turned to 180 degrees
- moved J12 1.78 mm to (150.4, 95.3)
- moved U5 1.55 mm to (148.3, 83.8)
- moved R31 1.32 mm to (135.9, 92.6)
- renumbered CH2_AC1 to locked
Connections:
- A1 pad 1: IN_CLOCK -> /MIDI_OUT
- A1 pad 11: unconnected-(A1-Pad11) -> /CLOCK_IN
Routing:
- net GND: track 48.5 -> 157.2 mm
- net IN_MIDI: track 15.5 -> 109.4 mm, vias 0 -> 3
- net Net-(D7-K): track 0.00 -> 65.3 mm, vias 0 -> 1
- net OUT_MIDI: track 0.00 -> 53.9 mm, vias 0 -> 2
- net IN_CLOCK: track 9.94 -> 59.0 mm
- net +5V: track 670.8 -> 711.3 mm, vias 0 -> 2
- net Net-(D7-A): track 0.00 -> 35.7 mm, vias 0 -> 2
- net /MIDI_OUT: track 0.00 -> 31.4 mm
- net SW_RESET: track 63.5 -> 79.8 mm
- net /CLOCK_IN: track 0.00 -> 15.6 mm
- net P_TEMPO: track 63.9 -> 74.8 mm
- net +12V: track 54.9 -> 65.3 mm
- net Net-(MIDI_OUT1-PadR): track 0.00 -> 8.54 mm
- net Net-(MIDI_IN1-PadR): track 0.00 -> 6.50 mm
- net LED_CLOCK: track 62.0 -> 57.4 mm
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Other:
- board size 164.6 x 108 mm -> 259.9 x 128.5 mm
- board text added: "RED!!"
- board text added: "SEMI-SENSIBLE SYNTH"
- board text added: "There are two large rectangles of F.Mask and B.Mask here to remove the front and back solder mask for a bare aluminium panel. If you are making an FR4 panel, remove these large rectangles to you get solder mask. If you want the symbols on the output jacks to be less visible (just 'embossed'), change them from F.Silkscreen to F.Cu (or try F.Mask). If you want the 'triggerspace' and 'semi-sensible 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"
- board text added: "locked"
- board text added: "triggerspace"
- board text removed: "+"
- board text removed: "Design/schematics based on Grids by Mutable-Instruments.net under a cc-by-sa 3.0 license."
- board text removed: "NanoGris V0.041.2 By Quinie"
- board text removed: "USB SIDE"
- board text removed: "this is NOT an orginal mutable instrument, much love for them though!"
