File: NanoGris.kicad_pcb (KiCad board)
At the start: 2 copper layers, 259.9 x 128.5 mm, 161 parts, among them J1 Conn_01x2, J10 Conn_01x12, J11 Conn_01x12, J12 Conn_02x05_Odd_Even, J13 Conn_01x10, J14 Conn_01x10, J15 Conn_01x10, J2 Conn_01x2, J3 Conn_01x2, J4 Conn_01x2, J7 Conn_01x10, Q1 2N3904, Q2 2N3904, U1 MCP6002_1, U2 MCP6002_1, U3 MCP6002_1, U4 L7805, U5 LM4040LP-5, U6 74HC595, U8 6N138, X1 CV_X, Y1 CV_Y

Commit message: Change MIDI ports to reuse clock out/rnd out ports.
Jumpers to select if we use MIDI or clock out / rnd.
Moved FILL knobs to a more ergonomic arrangement.
General polish to front panel.
Parts:
- removed CLK1: ClockOutput, Connector_Audio:Jack_3.5mm_QingPu_WQP-PJ398SM_Vertical_CircularHoles
- removed the H5 at (67.9, 52.8)
- removed the H5 at (52.1, 52.7)
- removed RND1: RandomGate, Connector_Audio:Jack_3.5mm_QingPu_WQP-PJ398SM_Vertical_CircularHoles
- added J4: Conn_01x4, Connector_PinHeader_2.54mm:PinHeader_1x04_P2.54mm_Vertical, B.Cu at (241.8, 114.9)
- added J5: Conn_01x3, Connector_PinHeader_2.54mm:PinHeader_1x03_P2.54mm_Vertical, B.Cu at (149.0, 120.6)
- added J6: Conn_01x3, Connector_PinHeader_2.54mm:PinHeader_1x03_P2.54mm_Vertical, B.Cu at (159.3, 120.6)
- added J8: Conn_01x3, Connector_PinHeader_2.54mm:PinHeader_1x03_P2.54mm_Vertical, B.Cu at (223.1, 114.9)
- C17, R47: moved to B.Cu
- J3: value Conn_01x2 -> Conn_01x4; footprint Connector_PinHeader_2.54mm:PinHeader_1x02_P2.54mm_Vertical -> Connector_PinHeader_2.54mm:PinHeader_1x04_P2.54mm_Vertical
- MIDI_IN_RND_OUT1: renamed from MIDI_IN1; value MIDI_IN -> MIDI_IN_RND
- MIDI_OUT_CLOCK_OUT1: renamed from MIDI_OUT1; value MIDI_OUT -> MIDI_OUT-CLOCK_OUT
- R49: moved to F.Cu
- moved R49 164.6 mm to (108.0, 113.1), turned to -90 degrees
- moved R47 91.9 mm to (246.1, 53.3), turned to 180 degrees
- moved J3 89.4 mm to (212.3, 103.5), turned to -90 degrees
- moved R50 79.3 mm to (203.2, 115.0), turned to 0 degrees
- moved MIDI_IN_RND_OUT1 67.5 mm to (214.4, 120.7), turned to -90 degrees
- moved MIDI_OUT_CLOCK_OUT1 66.3 mm to (214.4, 109.2), turned to -90 degrees
- moved P_CH1 31.6 mm to (227.9, 58.5)
- moved H23 31.3 mm to (37.2, 51.4)
- moved D7 29.0 mm to (259.0, 64.8), turned to 180 degrees
- moved C17 24.6 mm to (256.5, 47.0), turned to 180 degrees
- moved R48 23.5 mm to (249.0, 75.5)
- moved H17 20.1 mm to (54.2, 46.9)
- moved P_CH2 19.5 mm to (244.6, 70.5)
- moved H26 19.4 mm to (54.2, 63.4)
- moved D2 19.0 mm to (240.6, 88.5)
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Connections:
- J15 pad 7: CH_RND -> /MIDI_OUT-CLOCK_OUT
- J15 pad 8: CH_CLOCK -> /MIDI-IN_RND_OUT
- J3 pad 1: IN_MIDI -> GND
- J3 pad 2: OUT_MIDI -> Net-(J3-Pin_2)
- J7 pad 7: CH_RND -> /MIDI_OUT-CLOCK_OUT
- J7 pad 8: CH_CLOCK -> /MIDI-IN_RND_OUT
- MIDI_IN_RND_OUT1 pad R: Net-(MIDI_IN1-PadR) -> Net-(J4-Pin_3)
- MIDI_IN_RND_OUT1 pad S: unconnected-(MIDI_IN1-PadS) -> Net-(J4-Pin_2)
- MIDI_OUT_CLOCK_OUT1 pad R: Net-(MIDI_OUT1-PadR) -> Net-(J3-Pin_3)
- MIDI_OUT_CLOCK_OUT1 pad S: unconnected-(MIDI_OUT1-PadS) -> Net-(J3-Pin_2)
- MIDI_OUT_CLOCK_OUT1 pad T: Net-(MIDI_OUT1-PadT) -> /MIDI_OUT-CLOCK_OUT
- R47 pad 2: IN_MIDI -> Net-(J8-Pin_3)
- R48 pad 1: Net-(MIDI_IN1-PadR) -> Net-(J4-Pin_4)
- R49 pad 1: Net-(MIDI_OUT1-PadT) -> Net-(J6-Pin_1)
- R50 pad 2: Net-(MIDI_OUT1-PadR) -> Net-(J3-Pin_4)
- U8 pad 6: IN_MIDI -> Net-(J8-Pin_3)
Routing:
- net IN_MIDI: track 109.4 -> 206.4 mm
- net Net-(J8-Pin_3): track 0.00 -> 91.5 mm, vias 0 -> 1
- net OUT_MIDI: track 53.9 -> 133.4 mm, vias 2 -> 3
- net Net-(D7-A): track 35.7 -> 102.4 mm, vias 2 -> 0
- net /MIDI-IN_RND_OUT: track 0.00 -> 56.7 mm, vias 0 -> 1
- net Net-(J6-Pin_1): track 0.00 -> 54.8 mm
- net Net-(D7-K): track 65.3 -> 16.1 mm, vias 1 -> 0
- net GND: track 157.2 -> 110.8 mm
- net Net-(J4-Pin_4): track 0.00 -> 45.5 mm
- net Net-(J4-Pin_3): track 0.00 -> 33.2 mm
- net Net-(J4-Pin_2): track 0.00 -> 31.9 mm
- net CH_RND: track 48.1 -> 17.0 mm
- net Net-(J3-Pin_2): track 0.00 -> 24.9 mm
- net /MIDI_OUT-CLOCK_OUT: track 0.00 -> 21.8 mm
- net SW_RESET: track 79.8 -> 60.2 mm
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Other:
- board size 259.9 x 128.5 mm -> 257.6 x 128.5 mm
- board text removed: "RED!!"
- board text removed: "SEMI-SENSIBLE SYNTH"
- board text removed: "There are two large rectangles of F.Mask and B.Mask here to remove the front and back solder mask for a bare aluminium panel. If you are making an FR4 panel, remove these large rectangles to you get solder mask. If you want the symbols on the output jacks to be less visible (just 'embossed'), change them from F.Silkscreen to F.Cu (or try F.Mask). If you want the 'triggerspace' and 'semi-sensible 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"
- board text removed: "triggerspace"
