File: NanoGris.kicad_sch (KiCad schematic)
At the start: 112 parts, among them J10 Conn_01x12, J11 Conn_01x12, J12 Conn_02x05_Odd_Even, J13 Conn_01x10, J14 Conn_01x10, J15 Conn_01x10, J16 Conn_01x03, J7 Conn_01x10, Q1 2N3904, Q2 2N3904, U1 MCP6002_1, U2 MCP6002_1, U3 MCP6002_1, U4 L7805, U5 LM4040LP-5, U6 74HC595, X1 CV_X, Y1 CV_Y

Commit message: Updated with MIDI-TRS ports, numerous tweaks.
Moved front panel into main PCB design, remove old panels and gerbers that will no longer fit this design.
Parts:
- removed J16: Conn_01x03, Connector_PinHeader_2.54mm:PinHeader_1x03_P2.54mm_Vertical, symbol NanoGris-rescue:Conn_01x03-Connector_Generic-GridsNanoV3-rescue
- added C17: 100nf, Capacitor_THT:C_Disc_D5.0mm_W2.5mm_P2.50mm, symbol NanoGris-rescue:C-Device-GridsNanoV3-rescue
- added D7: 1n4148, Diode_THT:D_DO-34_SOD68_P7.62mm_Horizontal, symbol NanoGris-rescue:D-Device-GridsNanoV3-rescue
- added J1, J2, J4: Conn_01x2, Connector_PinSocket_2.54mm:PinSocket_1x02_P2.54mm_Vertical, symbol Connector_Generic:Conn_01x02
- added J3: Conn_01x2, Connector_PinHeader_2.54mm:PinHeader_1x02_P2.54mm_Vertical, symbol Connector_Generic:Conn_01x02
- added JP1, JP2: SolderJumper_2_Bridged, Jumper:SolderJumper-2_P1.3mm_Bridged_RoundedPad1.0x1.5mm, symbol Jumper:SolderJumper_2_Bridged
- added MIDI_IN1: MIDI_IN, Connector_Audio:Jack_3.5mm_QingPu_WQP-PJ398SM_Vertical_CircularHoles, symbol Connector_Audio:AudioJack3
- added MIDI_OUT1: MIDI_OUT, Connector_Audio:Jack_3.5mm_QingPu_WQP-PJ398SM_Vertical_CircularHoles, symbol Connector_Audio:AudioJack3
- added R46: 4.7k, Resistor_THT:R_Axial_DIN0204_L3.6mm_D1.6mm_P7.62mm_Horizontal, symbol NanoGris-rescue:R-Device-GridsNanoV3-rescue
- added R47, R48, R49, R50: 220, Resistor_THT:R_Axial_DIN0204_L3.6mm_D1.6mm_P7.62mm_Horizontal, symbol NanoGris-rescue:R-Device-GridsNanoV3-rescue
- added U8: 6N138, Package_DIP:DIP-8_W7.62mm_Socket_LongPads, symbol Isolator:6N138
- D5, D6: value 1n4148 -> 1N5817
- J10: symbol NanoGris-rescue:Conn_01x12-Connector_Generic-GridsNanoV3-rescue -> Connector_Generic:Conn_01x12
- J13, J14: symbol NanoGris-rescue:Conn_01x10-Connector_Generic-GridsNanoV3-rescue -> Connector_Generic:Conn_01x10
Connections:
- net +5V: now also C17.1, R47.1, R50.1, U8.8 (VCC)
- net GND: now also C17.2, R46.2, U8.5 (GND)
- net IN_CLOCK: now also J2.1 (Pin_1), JP2.1 (A); no longer A1.1 (D1/TX)
- net IN_MIDI: now also J3.1 (Pin_1), J4.1 (Pin_1), R47.2, U8.6 (VO2)
- net CLOCK_IN: now reaches A1.11 (D8)
- net CLOCK_IN: now also J1.1 (Pin_1), JP2.2 (B)
- new net: MIDI_OUT1.T, R49.1
- new net: MIDI_OUT1.R, R50.2
- new net: MIDI_IN1.R, R48.1
- new net: D7.2 (A), MIDI_IN1.T, U8.3 (C2)
- new net: D7.1 (K), R48.2, U8.2 (C1)
- new net: R46.1, U8.7 (VO1)
- new net MIDI_OUT: A1.1 (D1/TX), J2.2 (Pin_2), JP1.2 (B)
- new net OUT_MIDI: J1.2 (Pin_2), J3.2 (Pin_2), J4.2 (Pin_2), JP1.1 (A), R49.2
- no-connect marks 9 -> 10
Other:
- note added: "MIDI-TRS TYPE A"
- moved on the sheet: J13, J14
