File: NanoGris.kicad_sch (KiCad schematic)
At the start: 127 parts, among them J1 Conn_01x2, J10 Conn_01x12, J11 Conn_01x12, J12 Conn_02x05_Odd_Even, J13 Conn_01x10, J14 Conn_01x10, J15 Conn_01x10, J2 Conn_01x2, J3 Conn_01x2, J4 Conn_01x2, J7 Conn_01x10, Q1 2N3904, Q2 2N3904, U1 MCP6002_1, U2 MCP6002_1, U3 MCP6002_1, U4 L7805, U5 LM4040LP-5, U6 74HC595, U8 6N138, X1 CV_X, Y1 CV_Y

Commit message: Change MIDI ports to reuse clock out/rnd out ports.
Jumpers to select if we use MIDI or clock out / rnd.
Moved FILL knobs to a more ergonomic arrangement.
General polish to front panel.
Parts:
- removed CLK1: ClockOutput, Connector_Audio:Jack_3.5mm_QingPu_WQP-PJ398SM_Vertical_CircularHoles, symbol NanoGris-rescue:AudioJack2-Connector-GridsNanoV3-rescue
- removed J3: Conn_01x2, Connector_PinHeader_2.54mm:PinHeader_1x02_P2.54mm_Vertical, symbol Connector_Generic:Conn_01x02
- removed J4: Conn_01x2, Connector_PinSocket_2.54mm:PinSocket_1x02_P2.54mm_Vertical, symbol Connector_Generic:Conn_01x02
- removed RND1: RandomGate, Connector_Audio:Jack_3.5mm_QingPu_WQP-PJ398SM_Vertical_CircularHoles, symbol NanoGris-rescue:AudioJack2-Connector-GridsNanoV3-rescue
- added J3, J4: Conn_01x4, Connector_PinHeader_2.54mm:PinHeader_1x04_P2.54mm_Vertical, symbol Connector_Generic:Conn_01x04
- added J5, J6, J8: Conn_01x3, Connector_PinHeader_2.54mm:PinHeader_1x03_P2.54mm_Vertical, symbol Connector_Generic:Conn_01x03
- MIDI_IN_RND_OUT1: renamed from MIDI_IN1; value MIDI_IN -> MIDI_IN_RND
- MIDI_OUT_CLOCK_OUT1: renamed from MIDI_OUT1; value MIDI_OUT -> MIDI_OUT-CLOCK_OUT
Connections:
- net CH_CLOCK: now also J6.3 (Pin_3); no longer J15.8 (Pin_8), J7.8 (Pin_8)
- net CH_RND: now also J5.3 (Pin_3); no longer J15.7 (Pin_7), J7.7 (Pin_7)
- net GND: now also J3.1 (Pin_1), J4.1 (Pin_1)
- net IN_MIDI: now also J5.1 (Pin_1); no longer R47.2, U8.6 (VO2)
- net at R49.1: now also J6.1 (Pin_1); no longer MIDI_OUT_CLOCK_OUT1.T
- net at MIDI_OUT_CLOCK_OUT1.R: now also J3.3 (Pin_3); no longer R50.2
- net at MIDI_OUT_CLOCK_OUT1.S: now also J3.2 (Pin_2)
- net at MIDI_IN_RND_OUT1.R: now also J4.3 (Pin_3); no longer R48.1
- net at MIDI_IN_RND_OUT1.S: now also J4.2 (Pin_2)
- net at D7.2 (A), MIDI_IN_RND_OUT1.T, U8.3 (C2): now also J8.1 (Pin_1)
- new net: J3.4 (Pin_4), R50.2
- new net: J8.3 (Pin_3), R47.2, U8.6 (VO2)
- new net: J4.4 (Pin_4), R48.1
- new net MIDI-IN_RND_OUT: J15.8 (Pin_8), J5.2 (Pin_2), J7.8 (Pin_8), J8.2 (Pin_2)
- new net MIDI_OUT-CLOCK_OUT: J15.7 (Pin_7), J6.2 (Pin_2), J7.7 (Pin_7), MIDI_OUT_CLOCK_OUT1.T
- no-connect marks 10 -> 8
Other:
- note added: "For CLOCK-OUT, connect 1-2. For MIDI-OUT, connect 3-4."
- note added: "For MIDI-IN, connect 1-2. For RND-OUT, connect 2-3."
- note added: "For MIDI-OUT, connect 1-2. For CLOCK-OUT, connect 2-3."
- note added: "For RND-OUT, connect 1-2. For MIDI-IN, connect 2-3."
- note added: "For RND-OUT, connect 1-2. For MIDI-IN, connect 3-4."
- note added: "RING"
- note added: "TIP"
- moved on the sheet: C17, D7, H1, H2, J10, J11, J13, J14, J15, J7, MIDI_IN_RND_OUT1, MIDI_OUT_CLOCK_OUT1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
