File: triggerspace.kicad_pcb (KiCad board)
At the start: 2 copper layers, 257.6 x 128.5 mm, 161 parts, among them J1 Conn_01x2, J10 Conn_01x12, J11 Conn_01x12, J12 Conn_02x05_Odd_Even, J13 Conn_01x10, J14 Conn_01x10, J15 Conn_01x10, J2 Conn_01x2, J3 Conn_01x4, J4 Conn_01x2, J4 Conn_01x4, J5 Conn_01x3, J6 Conn_01x3, J7 Conn_01x10, J8 Conn_01x3, Q1 2N3904, Q2 2N3904, U1 MCP6002_1, U2 MCP6002_1, U3 MCP6002_1, U4 L7805, U5 LM4040LP-5, U6 74HC595, U8 6N138, X1 CV_X, Y1 CV_Y

Commit message: v0.042 release.
Update README with build notes.
Add schematic pdf.
KiCad files re-saved with version 8.0
Parts:
- renumbered locked to CH2_AC1
Other:
- board text added: "+"
- board text added: "."
- board text added: ".."
- board text added: "..."
- board text added: "5V"
- board text added: "ACC"
- board text added: "BUTTON_IN"
- board text added: "CHAOS"
- board text added: "CLK"
- board text added: "CLOCK"
- board text added: "CLOCK-OUT"
- board text added: "CLOCK_IN"
- board text added: "CV_CH1"
- board text added: "CV_CH2"
- board text added: "CV_CH3"
- board text added: "CV_RND"
- board text added: "CV_X"
- board text added: "CV_Y"
- board text added: "D0/RX"
- board text added: "D1/TX"
- board text added: "DENSITY"
- board text added: "Design/schematics based on Grids by Mutable-Instruments.net under a cc-by-sa 3.0 license."
- board text added: "FILL"
- board text added: "GND"
- board text added: "IF USING STOCK FIRMWARE CUT JP1 & JP2 BRIDGE JUMPER J1, J2"
- board text added: "JLCJLCJLCJLC"
- board text added: "LED_CH1"
- board text added: "LED_CH2"
- board text added: "LED_CH3"
- board text added: "LED_CLOCK"
- board text added: "Let's write a history book on a PCB ! Based on the original design by Émilie Gillet, 2012 (Mutable Instruments) Remixed to through-hole + Arduino Nano by Quinie, 2021 MIDI-In/Out jacks added by Andrew Perry, 2023 (semi-sensible synth) -> your modification log here <-"
- board text added: "MIDI-IN"
- board text added: "MIDI-OUT"
- board text added: "MIDI_IN"
- board text added: "MIDI_OUT"
- board text added: "MOSI"
- board text added: "NanoGris-MIDI V0.042"
- board text added: "OUTPUTS"
- board text added: "P_TEMPO"
- board text added: "RED!!"
- board text added: "RESET"
- board text added: "RESET_IN"
- board text added: "RND"
- board text added: "RND-OUT"
- board text added: "Remixed from the Mutable Instruments original by Quinie, 2021. MIDI in/out jacks added by Andrew Perry, 2023 (semi-sensible synth)."
- board text added: "SCK"
- board text added: "SEMI-SENSIBLE SYNTH"
- board text added: "SPEED"
- board text added: "SS"
- board text added: "TAP"
- board text added: "TRIG"
- board text added: "There are two large rectangles of F.Mask and B.Mask here to remove the front and back solder mask for a bare aluminium panel. If you are making an FR4 panel, remove these large rectangles to you get solder mask. If you want the symbols on the output jacks to be less visible (just 'embossed'), change them from F.Silkscreen to F.Cu (or try F.Mask). If you want the 'triggerspace' and 'semi-sensible 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"
- board text added: "USB SIDE"
- board text added: "X"
- board text added: "Y"
- board text added: "this is NOT an orginal mutable instrument, much love for them though!"
- board text added: "triggerspace"
- board text added: "{dblquote}triggerspace{dblquote}"
- board text removed: "locked"
