File: triggerspace.kicad_sch (KiCad schematic)
At the start: 128 parts, among them J1 Conn_01x2, J10 Conn_01x12, J11 Conn_01x12, J12 Conn_02x05_Odd_Even, J13 Conn_01x10, J14 Conn_01x10, J15 Conn_01x10, J2 Conn_01x2, J3 Conn_01x4, J4 Conn_01x4, J5 Conn_01x3, J6 Conn_01x3, J7 Conn_01x10, J8 Conn_01x3, Q1 2N3904, Q2 2N3904, U1 MCP6002_1, U2 MCP6002_1, U3 MCP6002_1, U4 L7805, U5 LM4040LP-5, U6 74HC595, U8 6N138, X1 CV_X, Y1 CV_Y

Commit message: Change naming to 'triggerspace' in most places
Other:
- company: (none) -> Andrew Perry (semi-sensible synth)
- title: NanoGris made from Mutable Instruments Grids -> triggerspace ("NanoGris-MIDI")
Changed lines of the file:
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@@
   (paper "A2")
   (title_block
-    (title "NanoGris made from Mutable Instruments Grids")
+    (title "triggerspace (\"NanoGris-MIDI\")")
     (date "2020-03-28")
-    (rev "0.41")
+    (rev "0.042")
+    (company "Andrew Perry (semi-sensible synth)")
   )
   (junction (at 245.11 57.15) (diameter 0) (color 0 0 0 0)
